File: PWRDBG/Hw/SAMM-FTPDB/POWER.kicad_sch (KiCad schematic)
At the start: 17 parts

Commit message: samm-ftpdb schematic
Parts:
- removed C?: 1uF, SAMPI:CAP0402, symbol SAMPI:CERCAP
- added BAT?: 3.2V/3.4Ah, symbol SAMPI:BATTERY
- added C?: 10uF, SAMPI:CAP0603, symbol SAMPI:CERCAP
- added R?: 10K@25°C, symbol SAMPI:NTC
- added U?: SCAP CHARGER, SAMPI:DFN3x3-10L, symbol SAMPI:LS0502SCD33S
- added U?: TPS63020, SAMPI:QFN14-EP-4X3, symbol Liem:TPS6302x
- F?: value 750mA -> 3A/6.3V
Connections:
- net +5V: now also U?.1 (VIN); no longer U?.1 (VIN), U?.2 (VIN), U?.3 (~{SHDN})
- net GND: now also BAT?.-, C?.1
- new net: U?.1 (VIN), U?.2 (VIN), U?.3 (~{SHDN})
- new net: BAT?.+, C?.2, U?.9 (VCAP)
Other:
- moved on the sheet: C?, D?, F?, J?, R?, TP?, U?
