File: FTDISWD/Design/SAMM-FTDISWD/FT4232.kicad_sch (KiCad schematic)
At the start: 30 parts

Commit message: SAMM-FTDISWD schematic update 2
Parts:
- removed D?: TRX2, Liem:LED0606_4P, symbol Liem:RB_LED
- removed R? (x2): 2.2K, Liem:RES0402, symbol My_Library:MOSFET_NCH
- removed U?: FT4232H, symbol SAMPI:FT4232H
- added C?: 100nF, Liem:CAP0402, symbol SAMPI:CERCAP
- added R?: 2.2K, Liem:RES0402, symbol SAMPI:RES
- added U?: FT2232H, SAMPI:VQFN-56_FTDI, symbol Liem:FT2232H
- C? (x2): value 22pF -> 8.2pF
- R? (x3): value 2.2K -> 1K; symbol My_Library:MOSFET_NCH -> SAMPI:RES
- R? (x3): symbol Triet_KiCAD_Sym:RES -> SAMPI:RES
- R?: symbol My_Library:MOSFET_NCH -> SAMPI:RES
- U?: value SPI EEPROM -> 93C46B
- Y?: value 12MHz -> 12MHz, CL=8pF
Connections:
- net +1V8: now also U?.2 (VCORE), U?.31 (VCORE), U?.43 (VREGOUT)
- net +3V3: now also R?.1, U?.16 (VCCIO), U?.36 (VCCIO), U?.44 (VREGIN), U?.50 (VCCIO)
- net GND: now also C?.1, U?.10 (TEST), U?.21 (GND), U?.41 (GND), U?.45 (GND), U?.57 (EP)
- net RXD1: now also U?.13 (ADBUS1/RXD/TDI/DO)
- net TXD1: now also U?.12 (ADBUS0/TXD/TCK/SK)
- net USB_N: now also U?.7 (DM)
- net USB_P: now also U?.8 (DP)
- net ~{RESET}: now also C?.2, R?.2, U?.11 (~{RESET})
- net at C?.2, C?.2, FT?.2: now also U?.9 (VPLL)
- net at C?.2, C?.2, FT?.2: now also U?.5 (VPHY)
- net at R?.1, U?.3 (DI): now also U?.55 (EEDATA)
- net at R?.2, U?.4 (CLK): now also U?.56 (EECLK)
- net at R?.2, U?.5 (CS): now also U?.1 (EECS)
- net at R?.1: now also D?.1 (GK); no longer D?.4 (RK)
- net at R?.2: now also U?.25 (ACBUS3/~{RXLED}/GPIOH3)
- net at R?.1: now also D?.4 (RK); no longer D?.1 (GK)
- net at R?.2: now also U?.26 (ACBUS4/~{TXLED}/GPIOH4)
- net at C?.2, Y?.1: now also U?.3 (OSCI)
- net at C?.2, Y?.3: now also U?.4 (OSCO)
- net at R?.2: now also U?.54 (~{PWREN})
- net at R?.2: now also U?.6 (REF)
- new net SWDIO_DIR: U?.37 (BDBUS4/~{DTR}/GPIOL0)
- new net SWD_EN: U?.38 (BDBUS5/~{DSR}/GPIOL1)
- new net TCK: U?.32 (BDBUS0/TXD/TCK/SK)
- new net TDI: U?.33 (BDBUS1/RXD/TDI/DO)
- new net TDO: U?.34 (BDBUS2/~{RTS}/TDO/DI)
- new net ~{TARGET_RESET}: U?.39 (BDBUS6/~{DCD}/GPIOL2)
- no-connect marks 25 -> 23
Other:
- note added: "Crystal Oscillator Load Capacitor Calculator https://www.electrocalc.dev/crystal-oscillator"
- moved on the sheet: C?, U?, Y?
